File: kicad_src/electronics_timer.kicad_sch (KiCad schematic)
At the start: 21 parts, among them U1 CD4013BE

Commit message: save progress, set up down in simple way done
Parts:
- added AFF1: LTS-6980HR, Display_7Segment:7SegmentLED_LTS6760_LTS6780, symbol Display_Character:LTS-6980HR
- added C3, C4: 1 uF, symbol Device:C_Small
- added DownBtn, UpBtn: SW_Push, symbol Switch:SW_Push
- added Q1: 2N3904, Package_TO_SOT_THT:TO-92_Inline, symbol Transistor_BJT:2N3904
- added R10, R12, R13, R8, R9: 1k Ohm, symbol Device:R_Small_US
- added R11: 220 Ohm, symbol Device:R_Small_US
- added U2: 40110, symbol 4xxx_IEEE:40110
- DefaultReset1: value 1000 nF -> 1 uF
Connections:
- net +9V: now also DefaultReset1.1, Reset1.1 (A), C3.1, C4.1, DownBtn.2, R12.1, R13.2, U2.16 (Vdd), UpBtn.2
- net GND: now also AFF1.5 (DP), Q1.1 (E), R10.2, R11.2, R8.2, R9.2, U2.10 (C), U2.4 (~{TE}), U2.6 (LE), U2.8 (Vss)
- net ResetButtonIn1: now also R8.1, U2.5 (CLR)
- new net: C4.2, DownBtn.1, R10.1, U2.7 (CKd)
- new net: C3.2, R9.1, U2.9 (CKu), UpBtn.1
- new net: Q1.3 (C), R13.1
- new net: AFF1.1 (e), U2.12 (Qe)
- new net: AFF1.10 (g), U2.2 (Qg)
- new net: AFF1.2 (d), U2.13 (Qd)
- new net: AFF1.4 (c), U2.14 (Qc)
- new net: AFF1.6 (b), U2.15 (Qb)
- new net: AFF1.7 (a), U2.1 (Qa)
- new net: AFF1.8 (C.K.), R11.1
- new net: AFF1.9 (f), U2.3 (Qf)
- new net: Q1.2 (B), U2.11 (B)
- new net CountStop: R12.2
Other:
- moved on the sheet: C1, C2, DefaultReset1, DefaultStop, MillisecondsC1, MillisecondsTimer1, OnOffA, PWR1, R1, R2, R3, R4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

Commit message: save progress
Parts:
- R12: value 1k Ohm -> 10k Ohm
Changed lines of the file:
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@@
 		(fields_autoplaced yes)
 		(property "Reference" "R12"
-			(at 226.06 151.1642 90)
+			(at 226.06 151.13 90)
 			(effects
 				(font
@@
 			)
 		)
-		(property "Value" "1k Ohm"
-			(at 226.06 153.7042 90)
+		(property "Value" "10k Ohm"
+			(at 226.06 153.67 90)
 			(effects
 				(font

Commit message: save progress
Parts:
- removed C3, C4: 1 uF, symbol Device:C_Small
- removed DefaultStop: 1000 nF, Capacitor_THT:CP_Radial_D8.0mm_P5.00mm, symbol Device:C
- removed Q1: 2N3904, Package_TO_SOT_THT:TO-92_Inline, symbol Transistor_BJT:2N3904
- removed R11: 220 Ohm, symbol Device:R_Small_US
- removed R12: 10k Ohm, symbol Device:R_Small_US
- removed R13, R2, R6, R7: 1k Ohm, symbol Device:R_Small_US
- removed R3: 1 kOhm, Resistor_THT:R_Axial_DIN0207_L6.3mm_D2.5mm_P10.16mm_Horizontal, symbol Device:R
- removed R5: 100k Ohm, Resistor_THT:R_Axial_DIN0207_L6.3mm_D2.5mm_P10.16mm_Horizontal, symbol Device:R
- removed RV1: R_Potentiometer_Trim, Potentiometer_THT:Potentiometer_Vishay_T73YP_Vertical, symbol Device:R_Potentiometer_Trim
- removed StartStop1: NE555P, Package_DIP:DIP-8_W7.62mm, symbol Timer:NE555P
- removed StartStopBtn1, UpBtn: SW_Push, symbol Switch:SW_Push
- removed StartStopLed1: LED, LED_THT:LED_D5.0mm, symbol Device:LED
- added C3, C4, C5, C6: 1 nF, Capacitor_THT:CP_Radial_D5.0mm_P2.50mm, symbol Device:C
- added C7: 10 nF, Capacitor_THT:CP_Radial_D5.0mm_P2.50mm, symbol Device:C
- added C8: 1 uF, Capacitor_THT:CP_Radial_D5.0mm_P2.50mm, symbol Device:C
- added D1, D2, D3, D4: D, symbol Device:D
- added OffSignal1, OffSignal2, OffSignal3: NE555P, Package_DIP:DIP-8_W7.62mm, symbol Timer:NE555P
- added OnOffBtn, UpBtn1: SW_Push, symbol Switch:SW_Push
- added R2, R6, R7: 10k Ohm, Resistor_THT:R_Axial_DIN0207_L6.3mm_D2.5mm_P10.16mm_Horizontal, symbol Device:R
- added R3, R5: 10k Ohm, symbol Device:R_Small_US
- R10, R8: value 1k Ohm -> 10k Ohm
- R9: value 1k Ohm -> 4.7k Ohm
- SecondsC1: renamed from MillisecondsC1; value 1000 nF -> 47 uF
- renumbered MillisecondsTimer1 to SecondsTimer1
Connections:
- net Start is gone; now on net GND: U1.1 (Q1)
- net GND: now also AFF1.8 (C.K.), U1.2 (*Q1), U1.3 (CLOCK1), U1.4 (RESET1), U1.5 (D1), C3.2, C4.2, C5.2, C6.2, C7.2, C8.2, OffSignal1.1 (GND), OffSignal2.1 (GND), OffSignal3.1 (GND), R3.2, R5.2; no longer R10.2, R9.2, U1.11 (CLOCK2), U1.12 (*Q2), U1.13 (Q2), U1.9 (D2)
- net ResetButtonIn1: no longer R8.1, U2.5 (CLR)
- net TimerPower1: now also U1.12 (*Q2), U1.9 (D2), OffSignal1.4 (R)
- net at DownBtn.1, U2.7 (CKd): now also D1.1 (K), R3.1; no longer R10.1
- net at SecondsC1.1, SecondsTimer1.2 (TR), SecondsTimer1.6 (THR): now also R2.2
- net at R4.2, SecondsTimer1.7 (DIS): now also R2.1
- net at R9.1: now also C8.1, D4.1 (K), OffSignal3.2 (TR), OffSignal3.6 (THR); no longer U2.9 (CKu)
- net at C2.2: now also R1.1, U1.11 (CLOCK2), D3.1 (K), OnOffBtn.1; no longer U1.3 (CLOCK1)
- net Borrow: now reaches U2.11 (B)
- net Borrow: now also OffSignal1.2 (TR), OffSignal2.2 (TR)
- net +9V renamed +5V
- net +5V: now also OffSignal1.8 (VCC), OffSignal2.4 (R), OffSignal2.8 (VCC), OnOffBtn.2, R6.2, R7.2; no longer DefaultReset1.1, DownBtn.2, Reset1.1 (A)
- net MilliSecondsPulse1 renamed SecondsPulse1
- net SecondsPulse1: now also D1.2 (A)
- removed net Stop: R1.1, U1.2 (*Q1), U1.5 (D1)
- new net: C4.1, OffSignal1.6 (THR), OffSignal1.7 (DIS), R6.1
- new net: D2.1 (K), DownBtn.2, UpBtn1.2
- new net: C3.1, OffSignal1.5 (CV)
- new net: R8.1, U2.5 (CLR)
- new net: C5.1, OffSignal2.5 (CV)
- new net: DefaultReset1.1, Reset1.1 (A)
- new net: C6.1, OffSignal2.6 (THR), OffSignal2.7 (DIS), R7.1
- new net: R5.1, U2.9 (CKu), UpBtn1.1
- new net: C7.1, OffSignal3.5 (CV)
- new net AlarmDischarge: D4.2 (A), OffSignal3.7 (DIS), R10.2, R9.2
- new net AlarmPower: OffSignal2.3 (Q), OffSignal3.4 (R), OffSignal3.8 (VCC), R10.1
- new net AlarmSignal: OffSignal3.3 (Q)
- new net OnOffSignal: D3.2 (A), OffSignal1.3 (Q)
- new net Q2: D2.2 (A), U1.13 (Q2)
Other:
- moved on the sheet: AFF1, C1, R4, R8, SecondsC1, SecondsTimer1, U1, U2

Commit message: chain counters
Parts:
- added C9: 100 uF, Capacitor_THT:CP_Radial_D5.0mm_P2.50mm, symbol Device:C
- added LS1: Speaker, symbol Device:Speaker
- added MinutesCounter1, MinutesDoubleCounter, SecundsDoubleCounter1: 40110, symbol 4xxx_IEEE:40110
- added MinutesDisplay1, MinutesDoubleDisplay1, SecondsDoubleDisplay1: LTS-6980HR, Display_7Segment:7SegmentLED_LTS6760_LTS6780, symbol Display_Character:LTS-6980HR
- renumbered AFF1 to SecondsDisplay, U2 to SecundsCounter
Connections:
- net +5V: now also MinutesCounter1.16 (Vdd), MinutesDoubleCounter.16 (Vdd), SecundsDoubleCounter1.16 (Vdd)
- net AlarmSignal: now also C9.2
- net GND: now also LS1.1, MinutesCounter1.4 (~{TE}), MinutesCounter1.6 (LE), MinutesCounter1.8 (Vss), MinutesDisplay1.5 (DP), MinutesDisplay1.8 (C.K.), MinutesDoubleCounter.4 (~{TE}), MinutesDoubleCounter.6 (LE), MinutesDoubleCounter.8 (Vss), MinutesDoubleDisplay1.5 (DP), MinutesDoubleDisplay1.8 (C.K.), SecondsDoubleDisplay1.5 (DP), SecondsDoubleDisplay1.8 (C.K.), SecundsDoubleCounter1.4 (~{TE}), SecundsDoubleCounter1.6 (LE), SecundsDoubleCounter1.8 (Vss); no longer SecundsCounter.10 (C)
- net Borrow renamed MinutesDoubleBorrow
- net MinutesDoubleBorrow: now also MinutesDoubleCounter.11 (B); no longer SecundsCounter.11 (B)
- new net: C9.1, LS1.2
- new net: MinutesDoubleCounter.12 (Qe), MinutesDoubleDisplay1.1 (e)
- new net: MinutesDoubleCounter.2 (Qg), MinutesDoubleDisplay1.10 (g)
- new net: MinutesDoubleCounter.13 (Qd), MinutesDoubleDisplay1.2 (d)
- new net: MinutesDoubleCounter.14 (Qc), MinutesDoubleDisplay1.4 (c)
- new net: MinutesDoubleCounter.15 (Qb), MinutesDoubleDisplay1.6 (b)
- new net: MinutesDoubleCounter.1 (Qa), MinutesDoubleDisplay1.7 (a)
- new net: MinutesDoubleCounter.3 (Qf), MinutesDoubleDisplay1.9 (f)
- new net: SecondsDoubleDisplay1.1 (e), SecundsDoubleCounter1.12 (Qe)
- new net: SecondsDoubleDisplay1.10 (g), SecundsDoubleCounter1.2 (Qg)
- new net: SecondsDoubleDisplay1.2 (d), SecundsDoubleCounter1.13 (Qd)
- new net: SecondsDoubleDisplay1.4 (c), SecundsDoubleCounter1.14 (Qc)
- new net: SecondsDoubleDisplay1.6 (b), SecundsDoubleCounter1.15 (Qb)
- new net: SecondsDoubleDisplay1.7 (a), SecundsDoubleCounter1.1 (Qa)
- new net: SecondsDoubleDisplay1.9 (f), SecundsDoubleCounter1.3 (Qf)
- new net: MinutesCounter1.12 (Qe), MinutesDisplay1.1 (e)
- new net: MinutesCounter1.2 (Qg), MinutesDisplay1.10 (g)
- new net: MinutesCounter1.13 (Qd), MinutesDisplay1.2 (d)
- new net: MinutesCounter1.14 (Qc), MinutesDisplay1.4 (c)
- new net: MinutesCounter1.15 (Qb), MinutesDisplay1.6 (b)
- new net: MinutesCounter1.1 (Qa), MinutesDisplay1.7 (a)
- new net: MinutesCounter1.3 (Qf), MinutesDisplay1.9 (f)
- new net DoubleSecondsBorrow: SecundsDoubleCounter1.11 (B)
- new net DoubleSecondsCarry: SecundsDoubleCounter1.10 (C)
- new net MinutesBorrow: MinutesCounter1.11 (B), MinutesDoubleCounter.7 (CKd)
- new net MinutesCarry: MinutesCounter1.10 (C), MinutesDoubleCounter.9 (CKu)
- new net MinutesDoubleCarry: MinutesDoubleCounter.10 (C)
- new net SecondsBorrow: SecundsCounter.11 (B), SecundsDoubleCounter1.7 (CKd)
- new net SecondsCarry: SecundsCounter.10 (C), SecundsDoubleCounter1.9 (CKu)
- new net SecondsDoubleBorrow: MinutesCounter1.7 (CKd)
- new net SecondsDoubleCarry: MinutesCounter1.9 (CKu)

Commit message: add reset button
Parts:
- removed R8: 10k Ohm, symbol Device:R_Small_US
- added R11: 10k Ohm, symbol Device:R_Small_US
Connections:
- net MinutesDoubleCarry is gone; now on net GND: MinutesDoubleCounter.10 (C)
- net +5V: now also DefaultReset1.1, Reset1.1 (A); no longer OffSignal2.4 (R)
- net GND: now also R11.2
- net ResetButtonIn1: now also MinutesCounter1.5 (CLR), MinutesDoubleCounter.5 (CLR), SecundsCounter.5 (CLR), SecundsDoubleCounter1.5 (CLR), R11.1
- net TimerPower1: now also OffSignal2.4 (R)
Other:
- note added: "We connect TimerPower1 to Reset to not trigger the 555 timer during counting down via button."
- moved on the sheet: DefaultReset1, Reset1

Commit message: save draft before rewrite
Parts:
- removed DownBtn: SW_Push, symbol Switch:SW_Push
- added DownBtn1: SW_Push, Button_Switch_THT:SW_PUSH_6mm, symbol Switch:SW_Push
- C1, C3, C4, C5, C6, C7, C8, C9: footprint Capacitor_THT:CP_Radial_D5.0mm_P2.50mm -> Capacitor_THT:CP_Radial_D8.0mm_P5.00mm
- C2: footprint (none) -> Capacitor_THT:CP_Radial_D8.0mm_P5.00mm
- D1, D2, D3, D4: footprint (none) -> Diode_THT:D_A-405_P10.16mm_Horizontal
- DefaultReset1: footprint Capacitor_THT:CP_Radial_D8.0mm_P5.00mm -> Capacitor_THT:CP_Radial_D5.0mm_P2.50mm
- LS1: footprint (none) -> Footprints:SpeakerConnector
- MinutesCounter1, SecundsDoubleCounter1: footprint (none) -> Package_DIP:DIP-16_W10.16mm
- MinutesDoubleCounter1: renamed from MinutesDoubleCounter; footprint (none) -> Package_DIP:DIP-16_W10.16mm
- OnOff1: renamed from OnOff; footprint slw-1678105:SW_SLW_1678105_DPDT_Slide -> Footprints:Big_Pwr_SWITCH
- OnOffBtn1: renamed from OnOffBtn; footprint (none) -> Button_Switch_THT:SW_PUSH_6mm
- R1, R10, R11, R3, R5, R9: footprint (none) -> Resistor_THT:R_Axial_DIN0207_L6.3mm_D2.5mm_P10.16mm_Horizontal
- SecundsCounter1: renamed from SecundsCounter; footprint (none) -> Package_DIP:DIP-16_W10.16mm
- U1: footprint N14 -> Package_DIP:DIP-14_W10.16mm
- UpBtn1: footprint (none) -> Button_Switch_THT:SW_PUSH_6mm
- renumbered OffSignal2 to AlarmPower1, OffSignal3 to AlarmSignal1, SecondsDisplay to SecondsDisplay1
Connections:
- net DoubleSecondsBorrow is gone; now on net SecondsDoubleBorrow: SecundsDoubleCounter1.11 (B)
- net DoubleSecondsCarry is gone; now on net SecondsDoubleCarry: SecundsDoubleCounter1.10 (C)
- net +5V: now also AlarmPower1.4 (R)
- net GND: now also SecundsCounter1.9 (CKu)
- net MinutesBorrow: now also R3.1, DownBtn1.1
- net MinutesCarry: now also R5.1, UpBtn1.1
- net TimerPower1: no longer AlarmPower1.4 (R)
- net at D2.1 (K), UpBtn1.2: now also DownBtn1.2
- net at D1.1 (K), SecundsCounter1.7 (CKd): no longer R3.1
