File: kicad_src/timer.kicad_sch (KiCad schematic)
At the start: 45 parts, among them U1 CD4013BE

Commit message: rewrite kicad schematics
Parts:
- removed AlarmPower1, OffSignal1, SecondsTimer1: NE555P, Package_DIP:DIP-8_W7.62mm, symbol Timer:NE555P
- removed C1: 1 nF, Capacitor_THT:CP_Radial_D8.0mm_P5.00mm, symbol Device:C
- removed MinutesCounter1, MinutesDoubleCounter1, SecundsCounter1, SecundsDoubleCounter1: 40110, Package_DIP:DIP-16_W10.16mm, symbol 4xxx_IEEE:40110
- removed MinutesDisplay1, MinutesDoubleDisplay1, SecondsDoubleDisplay1: LTS-6980HR, Display_7Segment:7SegmentLED_LTS6760_LTS6780, symbol Display_Character:LTS-6980HR
- removed OnOff1: SW_DPDT_x2, Footprints:Big_Pwr_SWITCH, symbol Switch:SW_DPDT_x2
- removed PWR1: Barrel_Jack, Connector_BarrelJack:BarrelJack_GCT_DCJ200-10-A_Horizontal, symbol Connector:Barrel_Jack
- removed R1: 1k Ohm, Resistor_THT:R_Axial_DIN0207_L6.3mm_D2.5mm_P10.16mm_Horizontal, symbol Device:R_Small_US
- removed R10, R11, R3, R5: 10k Ohm, Resistor_THT:R_Axial_DIN0207_L6.3mm_D2.5mm_P10.16mm_Horizontal, symbol Device:R_Small_US
- removed R2, R4, R6, R7: 10k Ohm, Resistor_THT:R_Axial_DIN0207_L6.3mm_D2.5mm_P10.16mm_Horizontal, symbol Device:R
- removed SecondsC1: 47 uF, Capacitor_THT:CP_Radial_D8.0mm_P5.00mm, symbol Device:C
- removed U1: CD4013BE, Package_DIP:DIP-14_W10.16mm, symbol CD4013BE:CD4013BE
- added AlarmPowerGenerator1, OnOffPulseGenerator1, SecondsPulseGenerator1: NE555P, Package_DIP:DIP-8_W7.62mm, symbol Timer:NE555P
- added C1: 1n, Capacitor_THT:CP_Radial_D5.0mm_P2.50mm, symbol Device:C_Small
- added DoubleMinutesCounter1, DoubleSecondsCounter1, MinutesCounter2, SecondsCounter1: 40110, Package_DIP:DIP-16_W10.16mm, symbol 4xxx_IEEE:40110
- added DoubleMinutesDisplay1, DoubleSecondsDisplay1, MinutesDisplay2: LTS-6980HR, Display_7Segment:7SegmentLED_LTS6760_LTS6780, symbol Display_Character:LTS-6980HR
- added J1: Barrel_Jack, Connector_BarrelJack:BarrelJack_GCT_DCJ200-10-A_Horizontal, symbol Connector:Barrel_Jack
- added OnOffBtnDefaultPress1: 1u, Capacitor_THT:CP_Radial_D5.0mm_P2.50mm, symbol Device:C_Small
- added OnOffLatch1: 4013, Package_DIP:DIP-14_W10.16mm, symbol 4xxx:4013
- added R1: 1k, Resistor_THT:R_Axial_DIN0207_L6.3mm_D2.5mm_P10.16mm_Horizontal, symbol Device:R_US
- added R10, R3, R4: 100k, Resistor_THT:R_Axial_DIN0207_L6.3mm_D2.5mm_P10.16mm_Horizontal, symbol Device:R_US
- added R11, R2, R5, R6: 10k, Resistor_THT:R_Axial_DIN0207_L6.3mm_D2.5mm_P10.16mm_Horizontal, symbol Device:R_US
- added R13, R7, R8: 10k Ohm, Resistor_THT:R_Axial_DIN0207_L6.3mm_D2.5mm_P10.16mm_Horizontal, symbol Device:R_Small_US
- added R14: 4.7k Ohm, Resistor_THT:R_Axial_DIN0207_L6.3mm_D2.5mm_P10.16mm_Horizontal, symbol Device:R_Small_US
- added SW3: PowerSwitch, Footprints:Big_Pwr_SWITCH, symbol Switch:SW_SPDT
- C2: value 1 uF -> 47u; footprint Capacitor_THT:CP_Radial_D8.0mm_P5.00mm -> Capacitor_THT:CP_Radial_D5.0mm_P2.50mm
- C3, C5, C7, C8, C9: footprint Capacitor_THT:CP_Radial_D8.0mm_P5.00mm -> Capacitor_THT:CP_Radial_D5.0mm_P2.50mm
- C4: value 1 nF -> 100u; footprint Capacitor_THT:CP_Radial_D8.0mm_P5.00mm -> Capacitor_THT:CP_Radial_D5.0mm_P2.50mm
- C6: value 1 nF -> 470u; footprint Capacitor_THT:CP_Radial_D8.0mm_P5.00mm -> Capacitor_THT:CP_Radial_D5.0mm_P2.50mm
- R9: value 4.7k Ohm -> 10k Ohm
Connections:
- net +5V: now also OnOffBtn1.1, AlarmPowerGenerator1.4 (R), AlarmPowerGenerator1.8 (VCC), DoubleMinutesCounter1.16 (Vdd), DoubleSecondsCounter1.16 (Vdd), J1.1, MinutesCounter2.16 (Vdd), OnOffBtnDefaultPress1.1, OnOffLatch1.14 (VDD), OnOffPulseGenerator1.8 (VCC), R11.2, R6.2, SecondsCounter1.16 (Vdd); no longer C2.1, OnOffBtn1.2
- net AlarmDischarge: now also R13.2, R14.2; no longer R9.2
- net AlarmPower: now also AlarmPowerGenerator1.3 (Q), R13.1
- net GND: now also C2.2, R9.2, AlarmPowerGenerator1.1 (GND), C1.2, DoubleMinutesCounter1.4 (~{TE}), DoubleMinutesCounter1.6 (LE), DoubleMinutesCounter1.8 (Vss), DoubleMinutesDisplay1.5 (DP), DoubleMinutesDisplay1.8 (C.K.), DoubleSecondsCounter1.4 (~{TE}), DoubleSecondsCounter1.6 (LE), DoubleSecondsCounter1.8 (Vss), DoubleSecondsDisplay1.5 (DP), DoubleSecondsDisplay1.8 (C.K.), MinutesCounter2.4 (~{TE}), MinutesCounter2.6 (LE), MinutesCounter2.8 (Vss), MinutesDisplay2.5 (DP), MinutesDisplay2.8 (C.K.), OnOffLatch1.10 (R), OnOffLatch1.11 (C), OnOffLatch1.4 (R), OnOffLatch1.6 (S), OnOffLatch1.7 (VSS), OnOffLatch1.8 (S), OnOffLatch1.9 (D), OnOffPulseGenerator1.1 (GND), R1.2, R10.1, R3.1, R4.1, R7.2, R8.2, SW3.3 (C), SecondsCounter1.4 (~{TE}), SecondsCounter1.6 (LE), SecondsCounter1.8 (Vss), SecondsCounter1.9 (CKu), SecondsPulseGenerator1.1 (GND)
- net OnOffSignal: now also OnOffPulseGenerator1.3 (Q)
- net ResetButtonIn1: now also DoubleMinutesCounter1.5 (CLR), DoubleSecondsCounter1.5 (CLR), MinutesCounter2.5 (CLR), R7.1, SecondsCounter1.5 (CLR)
- net at AlarmSignal1.2 (TR), AlarmSignal1.6 (THR), C8.1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: now also R14.1; no longer R9.1
- net at C4.1: now also OnOffPulseGenerator1.6 (THR), OnOffPulseGenerator1.7 (DIS), R6.1
- net at D1.1 (K): now also SecondsCounter1.7 (CKd)
- net at C3.1: now also OnOffPulseGenerator1.5 (CV)
- net at C5.1: now also AlarmPowerGenerator1.5 (CV)
- net at C6.1: now also AlarmPowerGenerator1.6 (THR), AlarmPowerGenerator1.7 (DIS), R11.1
- net at SecondsDisplay1.1 (e): now also SecondsCounter1.12 (Qe)
- net at SecondsDisplay1.10 (g): now also SecondsCounter1.2 (Qg)
- net at SecondsDisplay1.2 (d): now also SecondsCounter1.13 (Qd)
- net at SecondsDisplay1.4 (c): now also SecondsCounter1.14 (Qc)
- net at SecondsDisplay1.6 (b): now also SecondsCounter1.15 (Qb)
- net at SecondsDisplay1.7 (a): now also SecondsCounter1.1 (Qa)
- net at SecondsDisplay1.9 (f): now also SecondsCounter1.3 (Qf)
- net MinutesBorrow renamed MinutesCounterBorrow
- net MinutesCounterBorrow: now also DoubleMinutesCounter1.7 (CKd), MinutesCounter2.11 (B), R8.1
- net MinutesCarry renamed MinutesCounterCarry
- net MinutesCounterCarry: now also R9.1, DoubleMinutesCounter1.9 (CKu), MinutesCounter2.10 (C)
- net Q2 renamed UpDownBtnPower
- net UpDownBtnPower: now also OnOffLatch1.1 (Q)
- net SecondsPulse1 renamed SecondsPulseSignal
- net SecondsPulseSignal: now also SecondsPulseGenerator1.3 (Q)
- new net: D3.1 (K), OnOffBtn1.2, OnOffBtnDefaultPress1.2, OnOffLatch1.3 (C), R1.1
- new net: C2.1, R2.2, R5.1, R5.2, SecondsPulseGenerator1.2 (TR), SecondsPulseGenerator1.6 (THR), SecondsPulseGenerator1.7 (DIS)
- new net: DoubleSecondsCounter1.12 (Qe), DoubleSecondsDisplay1.1 (e)
- new net: DoubleSecondsCounter1.2 (Qg), DoubleSecondsDisplay1.10 (g)
- new net: DoubleSecondsCounter1.13 (Qd), DoubleSecondsDisplay1.2 (d)
- new net: DoubleSecondsCounter1.14 (Qc), DoubleSecondsDisplay1.4 (c)
- new net: DoubleSecondsCounter1.15 (Qb), DoubleSecondsDisplay1.6 (b)
- new net: DoubleSecondsCounter1.1 (Qa), DoubleSecondsDisplay1.7 (a)
- new net: DoubleSecondsCounter1.3 (Qf), DoubleSecondsDisplay1.9 (f)
- new net: J1.2, SW3.2 (B)
- new net: MinutesCounter2.1 (Qa), MinutesDisplay2.7 (a)
- new net: MinutesCounter2.12 (Qe), MinutesDisplay2.1 (e)
- new net: MinutesCounter2.13 (Qd), MinutesDisplay2.2 (d)
- new net: MinutesCounter2.14 (Qc), MinutesDisplay2.4 (c)
- new net: MinutesCounter2.15 (Qb), MinutesDisplay2.6 (b)
- new net: MinutesCounter2.2 (Qg), MinutesDisplay2.10 (g)
- new net: MinutesCounter2.3 (Qf), MinutesDisplay2.9 (f)
- new net: C1.1, SecondsPulseGenerator1.5 (CV)
- new net: OnOffLatch1.13 (Q), R3.2
- new net: OnOffLatch1.12 (~{Q}), R4.2
- new net: DoubleMinutesCounter1.12 (Qe), DoubleMinutesDisplay1.1 (e)
- new net: DoubleMinutesCounter1.2 (Qg), DoubleMinutesDisplay1.10 (g)
- new net: DoubleMinutesCounter1.13 (Qd), DoubleMinutesDisplay1.2 (d)
- new net: DoubleMinutesCounter1.14 (Qc), DoubleMinutesDisplay1.4 (c)
- new net: DoubleMinutesCounter1.15 (Qb), DoubleMinutesDisplay1.6 (b)
- new net: DoubleMinutesCounter1.1 (Qa), DoubleMinutesDisplay1.7 (a)
- new net: DoubleMinutesCounter1.3 (Qf), DoubleMinutesDisplay1.9 (f)
- new net: DoubleMinutesCounter1.10 (C), R10.2
- new net DoubleMinutesCounterBorrow: AlarmPowerGenerator1.2 (TR), DoubleMinutesCounter1.11 (B), OnOffPulseGenerator1.2 (TR)
- new net DoubleSecondsCounterBorrow: DoubleSecondsCounter1.11 (B), MinutesCounter2.7 (CKd)
- new net DoubleSecondsCounterCarry: DoubleSecondsCounter1.10 (C), MinutesCounter2.9 (CKu)
- new net SecondsCounterBorrow: DoubleSecondsCounter1.7 (CKd), SecondsCounter1.11 (B)
- new net SecondsCounterCarry: DoubleSecondsCounter1.9 (CKu), SecondsCounter1.10 (C)
- new net SecondsPulsePower: OnOffLatch1.2 (~{Q}), OnOffLatch1.5 (D), OnOffPulseGenerator1.4 (R), R2.1, SecondsPulseGenerator1.4 (R), SecondsPulseGenerator1.8 (VCC)
- no-connect marks 0 -> 5
Other:
- note added: "We connect SecondsPuslsePower to Reset to not trigger the 555 timer during counting down via button."
- note removed: "We connect TimerPower1 to Reset to not trigger the 555 timer during counting down via button."
